File: agv-skladiscni-v1/agv-skladiscni-v5.sch (KiCad schematic (older format))
At the start: 56 parts, among them IC1 NLAST4051DTR2G, IC2 NLAST4051DTR2G, J1 TOF_0, J2 TOF_1, J3 GP1, J4 I2C, J5 ADC, J6 GP0, Q1 BSS138, Q2 BSS138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

Commit message: changed to Velocity PID with FeedForward
Parts:
- IC1, IC2: symbol agv-skladiscni-v1-rescue:NLAST4051DTR2G-NLAST4051DTR2G -> agv-skladiscni-v5-rescue:NLAST4051DTR2G-NLAST4051DTR2G-agv-skladiscni-v1-rescue
Changed lines of the file:
@@
 EESchema Schematic File Version 4
-LIBS:agv-skladiscni-v1-cache
+LIBS:agv-skladiscni-v5-cache
 EELAYER 26 0
 EELAYER END
@@
 	9000 2150 8950 2150
 $Comp
-L agv-skladiscni-v1-rescue:NLAST4051DTR2G-NLAST4051DTR2G IC1
+L agv-skladiscni-v5-rescue:NLAST4051DTR2G-NLAST4051DTR2G-agv-skladiscni-v1-rescue IC1
 U 1 1 5BECC76D
 P 8600 3200
@@
 	10000 3800 9900 3800
 $Comp
-L agv-skladiscni-v1-rescue:NLAST4051DTR2G-NLAST4051DTR2G IC2
+L agv-skladiscni-v5-rescue:NLAST4051DTR2G-NLAST4051DTR2G-agv-skladiscni-v1-rescue IC2
 U 1 1 5C03A0C5
 P 8600 4750
